File: pcb/stm32_uc.kicad_sch (KiCad schematic)
At the start: 28 parts

Commit message: moved schematic/pcb files
Parts:
- C1, C2: renamed from C?; footprint (none) -> Capacitor_SMD:C_0805_2012Metric
- C10, C11, C12, C13, C4, C5, C6, C7, C9: renamed from C?; footprint (none) -> Capacitor_SMD:C_0402_1005Metric
- C3, C8: renamed from C?; footprint (none) -> Capacitor_SMD:C_0603_1608Metric
- D1: renamed from D?; footprint (none) -> LED_SMD:LED_0603_1608Metric
- FB1: renamed from FB?; footprint (none) -> Inductor_SMD:L_0603_1608Metric
- J1, J2: renamed from J?; footprint (none) -> Connector_PinHeader_2.54mm:PinHeader_1x18_P2.54mm_Vertical
- J3: renamed from J?; footprint (none) -> Connector_USB:USB_C_Receptacle_GCT_USB4085
- J4: renamed from J?; footprint (none) -> Connector_PinHeader_2.54mm:PinHeader_1x04_P2.54mm_Vertical
- R1, R2, R3, R4, R5: renamed from R?; footprint (none) -> Resistor_SMD:R_0402_1005Metric
- SW1: renamed from SW?; footprint (none) -> Button_Switch_THT:SW_E-Switch_EG1224_SPDT_Angled
- Y1: renamed from Y?; footprint (none) -> Crystal:Crystal_SMD_3225-4Pin_3.2x2.5mm
- gave numbers to parts that had none: 2
Connections:
- net +3V3: no longer J2.3 (Pin_3), U2.2 (PC13)
- new net PC13: J2.3 (Pin_3), U2.2 (PC13)
Other:
- note added: "1x 100nF per VDD pin"
- note added: "5k1 resistors in both CC, sets up USB-c in usb 2.0 mode"
- note added: "CL=2*(CL0-Cs)=2*(10p-5p)=10pF"
- note added: "Microcontroller"
- note added: "Pin Headers"
- note added: "Pin-out using STM32CubeIDE"
- note added: "Power Supply"
- note added: "STM32F103_ucboard"
- note added: "USB"
- note added: "USB App note AN4879"
- note added: "VBus comes from USB (nom. +5V). Min. 22uF inp.outp. caps"
- note added: "VDDA Filtering"
- company: (none) -> jpais
- title: (none) -> STM32f103_ucboard
- moved on the sheet: C1, C10, C11, C12, C13, C2, C3, C4, C5, C6, C7, C8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

Commit message: fix pin header pinout
Parts:
- C8: footprint Capacitor_SMD:C_0603_1608Metric -> Capacitor_SMD:C_0402_1005Metric
Connections:
- net PA0: now also J1.17 (Pin_17); no longer J1.7 (Pin_7)
- net PA1: now also J1.16 (Pin_16); no longer J1.8 (Pin_8)
- net PA15: no longer J1.17 (Pin_17)
- net PA2: now also J1.15 (Pin_15); no longer J1.9 (Pin_9)
- net PA3: now also J1.14 (Pin_14); no longer J1.10 (Pin_10)
- net PA4: now also J1.13 (Pin_13); no longer J1.11 (Pin_11)
- net PA6: now also J1.11 (Pin_11); no longer J1.13 (Pin_13)
- net PA7: now also J1.10 (Pin_10); no longer J1.14 (Pin_14)
- net PA8: now also J2.4 (Pin_4); no longer J1.15 (Pin_15)
- net PA9: now also J2.5 (Pin_5); no longer J1.16 (Pin_16)
- net PB0: now also J1.9 (Pin_9); no longer J2.6 (Pin_6)
- net PB1: now also J1.8 (Pin_8); no longer J2.7 (Pin_7)
- net PB10: now also J1.6 (Pin_6); no longer J2.16 (Pin_16)
- net PB11: now also J1.5 (Pin_5); no longer J1.2 (Pin_2)
- net PB12: now also J1.4 (Pin_4); no longer J1.3 (Pin_3)
- net PB13: now also J1.3 (Pin_3); no longer J1.4 (Pin_4)
- net PB14: now also J1.2 (Pin_2); no longer J1.5 (Pin_5)
- net PB15: now also J2.3 (Pin_3); no longer J1.6 (Pin_6)
- net PB2: now also J1.7 (Pin_7); no longer J2.8 (Pin_8)
- net PB3: now also J2.6 (Pin_6); no longer J2.9 (Pin_9)
- net PB4: now also J2.7 (Pin_7); no longer J2.10 (Pin_10)
- net PB5: now also J2.8 (Pin_8); no longer J2.11 (Pin_11)
- net PB6: now also J2.9 (Pin_9); no longer J2.12 (Pin_12)
- net PB7: now also J2.10 (Pin_10); no longer J2.13 (Pin_13)
- net PB8: now also J2.11 (Pin_11); no longer J2.14 (Pin_14)
- net PB9: now also J2.12 (Pin_12); no longer J2.15 (Pin_15)
- net PC13: now also J2.14 (Pin_14); no longer J2.3 (Pin_3)
- net PC14: now also J2.15 (Pin_15); no longer J2.4 (Pin_4)
- net PC15: now also J2.16 (Pin_16); no longer J2.5 (Pin_5)
- net USB_D+: now also J3.A6 (D+), J3.B6 (D+), R3.2
- net USB_D-: now also J3.A7 (D-), J3.B7 (D-)
Changed lines of the file:
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@@
     (effects (font (size 2 2) (thickness 0.4) bold) (justify left bottom))
   )
+  (label "PA6" (at 259.08 100.33 0)
+    (effects (font (size 1.27 1.27)) (justify left bottom))
+  )
   (label "PC15" (at 132.08 187.96 0)
     (effects (font (size 1.27 1.27)) (justify left bottom))
@@
     (effects (font (size 1.27 1.27)) (justify left bottom))
   )
-  (label "PB9" (at 306.07 110.49 180)
+  (label "PA4" (at 259.08 105.41 0)
+    (effects (font (size 1.27 1.27)) (justify left bottom))
+  )
+  (label "PB9" (at 306.07 102.87 180)
     (effects (font (size 1.27 1.27)) (justify right bottom))
   )
@@
     (effects (font (size 1.27 1.27)) (justify left bottom))
   )
-  (label "PA1" (at 259.08 92.71 0)
-    (effects (font (size 1.27 1.27)) (justify left bottom))
-  )
-  (label "PB0" (at 306.07 87.63 180)
-    (effects (font (size 1.27 1.27)) (justify right bottom))
-  )
-  (label "PA8" (at 259.08 110.49 0)
-    (effects (font (size 1.27 1.27)) (justify left bottom))
-  )
   (label "PA9" (at 177.8 215.9 180)
     (effects (font (size 1.27 1.27)) (justify right bottom))
   )
-  (label "PC13" (at 306.07 80.01 180)
-    (effects (font (size 1.27 1.27)) (justify right bottom))
-  )
-  (label "PA6" (at 259.08 105.41 0)
+  (label "PC13" (at 306.07 107.95 180)
+    (effects (font (size 1.27 1.27)) (justify right bottom))
+  )
+  (label "PB4" (at 132.08 203.2 0)
+    (effects (font (size 1.27 1.27)) (justify left bottom))
+  )
+  (label "PB12" (at 259.08 82.55 0)
+    (effects (font (size 1.27 1.27)) (justify left bottom))
+  )
+  (label "PA3" (at 259.08 107.95 0)
+    (effects (font (size 1.27 1.27)) (justify left bottom))
+  )
+  (label "USB_D+" (at 252.73 179.07 180)
+    (effects (font (size 1.27 1.27)) (justify right bottom))
+  )
+  (label "PA8" (at 306.07 82.55 180)
+    (effects (font (size 1.27 1.27)) (justify right bottom))
+  )
+  (label "CC1" (at 288.29 163.83 0)
     (effects (font (size 1.27 1.27)) (justify left bottom))
   )
@@
     (effects (font (size 1.27 1.27)) (justify left bottom))
   )
-  (label "PB4" (at 132.08 203.2 0)
-    (effects (font (size 1.27 1.27)) (justify left bottom))
-  )
-  (label "PB1" (at 306.07 90.17 180)
-    (effects (font (size 1.27 1.27)) (justify right bottom))
-  )
-  (label "PA2" (at 259.08 95.25 0)
-    (effects (font (size 1.27 1.27)) (justify left bottom))
-  )
-  (label "PB2" (at 306.07 92.71 180)
-    (effects (font (size 1.27 1.27)) (justify right bottom))
-  )
-  (label "CC1" (at 288.29 163.83 0)
-    (effects (font (size 1.27 1.27)) (justify left bottom))
-  )
   (label "PA15" (at 177.8 231.14 180)
     (effects (font (size 1.27 1.27)) (justify right bottom))
   )
-  (label "PB14" (at 259.08 85.09 0)
-    (effects (font (size 1.27 1.27)) (justify left bottom))
-  )
   (label "USB_D-" (at 181.61 220.98 180)
     (effects (font (size 1.27 1.27)) (justify right bottom))
@@
     (effects (font (size 1.27 1.27)) (justify left bottom))
   )
+  (label "PB2" (at 259.08 90.17 0)
+    (effects (font (size 1.27 1.27)) (justify left bottom))
+  )
   (label "PA0" (at 177.8 193.04 180)
     (effects (font (size 1.27 1.27)) (justify right bottom))
@@
     (effects (font (size 1.27 1.27)) (justify right bottom))
   )
+  (label "PB1" (at 259.08 92.71 0)
+    (effects (font (size 1.27 1.27)) (justify left bottom))
+  )
   (label "BOOT0" (at 132.08 170.18 0)
     (effects (font (size 1.27 1.27)) (justify left bottom))
@@
     (effects (font (size 1.27 1.27)) (justify right bottom))
   )
-  (label "PB11" (at 259.08 77.47 0)
+  (label "PB0" (at 259.08 95.25 0)
+    (effects (font (size 1.27 1.27)) (justify left bottom))
+  )
+  (label "PA0" (at 259.08 115.57 0)
     (effects (font (size 1.27 1.27)) (justify left bottom))
   )
@@
     (effects (font (size 1.27 1.27)) (justify left bottom))
   )
+  (label "USB_D-" (at 252.73 176.53 180)
+    (effects (font (size 1.27 1.27)) (justify right bottom))
+  )
   (label "PC14" (at 132.08 185.42 0)
     (effects (font (size 1.27 1.27)) (justify left bottom))
   )
-  (label "PB15" (at 259.08 87.63 0)
-    (effects (font (size 1.27 1.27)) (justify left bottom))
-  )
   (label "PA7" (at 177.8 210.82 180)
     (effects (font (size 1.27 1.27)) (justify right bottom))
   )
-  (label "PA7" (at 259.08 107.95 0)
-    (effects (font (size 1.27 1.27)) (justify left bottom))
-  )
-  (label "PA4" (at 259.08 100.33 0)
+  (label "PA2" (at 259.08 110.49 0)
     (effects (font (size 1.27 1.27)) (justify left bottom))
   )
@@
     (effects (font (size 0.5 0.5)) (justify left bottom))
   )
-  (label "PB6" (at 306.07 102.87 180)
+  (label "PB6" (at 306.07 95.25 180)
     (effects (font (size 1.27 1.27)) (justify right bottom))
   )
@@
     (effects (font (size 1.27 1.27)) (justify left bottom))
   )
-  (label "PB13" (at 259.08 82.55 0)
+  (label "PB13" (at 259.08 80.01 0)
     (effects (font (size 1.27 1.27)) (justify left bottom))
   )
@@
     (effects (font (size 1.27 1.27)) (justify left bottom))
   )
-  (label "PB12" (at 259.08 80.01 0)
-    (effects (font (size 1.27 1.27)) (justify left bottom))
-  )
-  (label "PA3" (at 259.08 97.79 0)
-    (effects (font (size 1.27 1.27)) (justify left bottom))
-  )
   (label "PB7" (at 132.08 210.82 0)
     (effects (font (size 1.27 1.27)) (justify left bottom))
   )
-  (label "PA9" (at 259.08 113.03 0)
-    (effects (font (size 1.27 1.27)) (justify left bottom))
-  )
-  (label "PB4" (at 306.07 97.79 180)
+  (label "PB4" (at 306.07 90.17 180)
     (effects (font (size 1.27 1.27)) (justify right bottom))
   )
@@
     (effects (font (size 1.27 1.27)) (justify right bottom))
   )
-  (label "PB5" (at 306.07 100.33 180)
-    (effects (font (size 1.27 1.27)) (justify right bottom))
+  (label "PB5" (at 306.07 92.71 180)
+    (effects (font (size 1.27 1.27)) (justify right bottom))
+  )
+  (label "PA1" (at 259.08 113.03 0)
+    (effects (font (size 1.27 1.27)) (justify left bottom))
   )
   (label "PB5" (at 132.08 205.74 0)
     (effects (font (size 1.27 1.27)) (justify left bottom))
   )
-  (label "PC14" (at 306.07 82.55 180)
-    (effects (font (size 1.27 1.27)) (justify right bottom))
-  )
-  (label "PB3" (at 306.07 95.25 180)
-    (effects (font (size 1.27 1.27)) (justify right bottom))
-  )
-  (label "PB7" (at 306.07 105.41 180)
+  (label "PB14" (at 259.08 77.47 0)
+    (effects (font (size 1.27 1.27)) (justify left bottom))
+  )
+  (label "PC14" (at 306.07 110.49 180)
+    (effects (font (size 1.27 1.27)) (justify right bottom))
+  )
+  (label "PB3" (at 306.07 87.63 180)
+    (effects (font (size 1.27 1.27)) (justify right bottom))
+  )
+  (label "PB7" (at 306.07 97.79 180)
+    (effects (font (size 1.27 1.27)) (justify right bottom))
+  )
+  (label "PB15" (at 306.07 80.01 180)
     (effects (font (size 1.27 1.27)) (justify right bottom))
   )
@@
     (effects (font (size 1.27 1.27)) (justify right bottom))
   )
-  (label "PA0" (at 259.08 90.17 0)
-    (effects (font (size 1.27 1.27)) (justify left bottom))
-  )
-  (label "PB8" (at 306.07 107.95 180)
-    (effects (font (size 1.27 1.27)) (justify right bottom))
-  )
-  (label "HSE_OUT" (at 115.57 209.55 90)
-    (effects (font (size 1.27 1.27)) (justify left bottom))
-  )
-  (label "PC15" (at 306.07 85.09 180)
+  (label "PB8" (at 306.07 100.33 180)
+    (effects (font (size 1.27 1.27)) (justify right bottom))
+  )
+  (label "PA7" (at 259.08 97.79 0)
+    (effects (font (size 1.27 1.27)) (justify left bottom))
+  )
+  (label "HSE_OUT" (at 115.57 200.66 270)
+    (effects (font (size 1.27 1.27)) (justify right bottom))
+  )
+  (label "PC15" (at 306.07 113.03 180)
     (effects (font (size 1.27 1.27)) (justify right bottom))
   )
@@
     (effects (font (size 1.27 1.27)) (justify right bottom))
   )
-  (label "HSE_IN" (at 92.71 209.55 90)
-    (effects (font (size 1.27 1.27)) (justify left bottom))
+  (label "PA9" (at 306.07 85.09 180)
+    (effects (font (size 1.27 1.27)) (justify right bottom))
+  )
+  (label "HSE_IN" (at 92.71 200.66 270)
+    (effects (font (size 1.27 1.27)) (justify right bottom))
   )
   (label "USB_D+" (at 181.61 223.52 180)
     (effects (font (size 1.27 1.27)) (justify right bottom))
   )
+  (label "PB11" (at 259.08 85.09 0)
+    (effects (font (size 1.27 1.27)) (justify left bottom))
+  )
   (label "PA3" (at 177.8 200.66 180)
     (effects (font (size 1.27 1.27)) (justify right bottom))
@@
     (effects (font (size 1.27 1.27)) (justify left bottom))
   )
-  (label "PB10" (at 306.07 113.03 180)
-    (effects (font (size 1.27 1.27)) (justify right bottom))
+  (label "PB10" (at 259.08 87.63 0)
+    (effects (font (size 1.27 1.27)) (justify left bottom))
   )
   (label "SWCLK" (at 181.61 228.6 180)
@@
   )
   (label "HSE_OUT" (at 129.54 177.8 0)
-    (effects (font (size 1.27 1.27)) (justify left bottom))
-  )
-  (label "PA15" (at 259.08 115.57 0)
     (effects (font (size 1.27 1.27)) (justify left bottom))
   )
@@
       (effects (font (size 1.27 1.27)) (justify left))
     )
-    (property "Footprint" "Capacitor_SMD:C_0603_1608Metric" (id 2) (at 174.9552 151.13 0)
+    (property "Footprint" "Capacitor_SMD:C_0402_1005Metric" (id 2) (at 174.9552 151.13 0)
       (effects (font (size 1.27 1.27)) hide)
     )
@@
     )
     (path "/c18c9479-eadf-421e-9d53-4c7649991dae"
-      (reference "C8") (unit 1) (value "10n") (footprint "Capacitor_SMD:C_0603_1608Metric")
+      (reference "C8") (unit 1) (value "10n") (footprint "Capacitor_SMD:C_0402_1005Metric")
     )
     (path "/6c899590-b6d7-4f13-bd8a-ec867ec66659"

Commit message: fix
Parts:
- SW1: footprint Button_Switch_THT:SW_E-Switch_EG1224_SPDT_Angled -> Button_Switch_SMD:SW_SPDT_PCM12
Changed lines of the file:
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@@
     (property "Reference" "SW1" (id 0) (at 116.84 167.64 0))
     (property "Value" "SW_SPDT" (id 1) (at 115.57 175.26 0))
-    (property "Footprint" "Button_Switch_THT:SW_E-Switch_EG1224_SPDT_Angled" (id 2) (at 114.3 170.18 0)
+    (property "Footprint" "Button_Switch_SMD:SW_SPDT_PCM12" (id 2) (at 114.3 170.18 0)
       (effects (font (size 1.27 1.27)) hide)
     )
@@
     )
     (path "/aa7aec69-26d5-49c4-aa8f-2811432a1bd2"
-      (reference "SW1") (unit 1) (value "SW_SPDT") (footprint "Button_Switch_THT:SW_E-Switch_EG1224_SPDT_Angled")
+      (reference "SW1") (unit 1) (value "SW_SPDT") (footprint "Button_Switch_SMD:SW_SPDT_PCM12")
     )
     (path "/36fe1a76-d2e1-4616-ae7c-c8bcfa6a8eec"

Commit message: finished rough layout
Parts:
- added H1, H2, H3, H4: MountingHole, MountingHole:MountingHole_2.2mm_M2, symbol Mechanical:MountingHole
Other:
- note added: "M2"
- note added: "Mounting Holes"
Changed lines of the file:
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@@
+    (stroke (width 0) (type default) (color 0 0 0 0))
+  )
+  (polyline (pts (xy 250.19 224.79) (xy 250.19 250.19))
     (stroke (width 0) (type default) (color 0 0 0 0))
   )
@@
     (stroke (width 0) (type default) (color 0 0 0 0))
   )
+  (polyline (pts (xy 276.86 250.19) (xy 250.19 250.19))
+    (stroke (width 0) (type default) (color 0 0 0 0))
+  )
   (wire (pts (xy 259.08 110.49) (xy 266.7 110.49))
     (stroke (width 0) (type default) (color 0 0 0 0))
@@
     (stroke (width 0) (type default) (color 0 0 0 0))
   )
+  (polyline (pts (xy 276.86 224.79) (xy 276.86 250.19))
+    (stroke (width 0) (type default) (color 0 0 0 0))
+  )
   (wire (pts (xy 292.1 177.8) (xy 288.29 177.8))
     (stroke (width 0) (type default) (color 0 0 0 0))
@@
   )
   (polyline (pts (xy 82.55 57.15) (xy 152.4 57.15))
+    (stroke (width 0) (type default) (color 0 0 0 0))
+  )
+  (polyline (pts (xy 250.19 224.79) (xy 276.86 224.79))
     (stroke (width 0) (type default) (color 0 0 0 0))
   )
@@
     (effects (font (size 1.27 1.27)) (justify left bottom))
   )
+  (text "Mounting Holes" (at 250.19 223.52 0)
+    (effects (font (size 2 2) (thickness 0.47) bold) (justify left bottom))
+  )
   (text "Pin-out using STM32CubeIDE\n" (at 82.55 260.35 0)
     (effects (font (size 1.27 1.27)) (justify left bottom))
@@
   )
   (text "VDDA Filtering" (at 187.96 162.56 0)
+    (effects (font (size 1.27 1.27)) (justify left bottom))
+  )
+  (text "M2\n" (at 250.19 254 0)
     (effects (font (size 1.27 1.27)) (justify left bottom))
   )
@@
     )
     (pin "1")
+  )
+  (symbol (lib_id "Mechanical:MountingHole") (at 257.81 240.03 0) (unit 1)
+    (in_bom yes) (on_board yes)
+    (property "Reference" "H3" (id 0) (at 252.73 240.03 0)
+      (effects (font (size 1.27 1.27)) (justify left))
+    )
+    (property "Value" "MountingHole" (id 1) (at 260.35 240.03 0)
+      (effects (font (size 1.27 1.27)) (justify left))
+    )
+    (property "Footprint" "MountingHole:MountingHole_2.2mm_M2" (id 2) (at 257.81 240.03 0)
+      (effects (font (size 1.27 1.27)) hide)
+    )
+    (property "Datasheet" "~" (id 3) (at 257.81 240.03 0)
+      (effects (font (size 1.27 1.27)) hide)
+    )
   )
   (symbol (lib_id "Device:C") (at 135.89 147.32 0) (unit 1)
@@
     )
     (pin "1")
+  )
+  (symbol (lib_id "Mechanical:MountingHole") (at 257.81 234.95 0) (unit 1)
+    (in_bom yes) (on_board yes)
+    (property "Reference" "H2" (id 0) (at 252.73 234.95 0)
+      (effects (font (size 1.27 1.27)) (justify left))
+    )
+    (property "Value" "MountingHole" (id 1) (at 260.35 234.95 0)
+      (effects (font (size 1.27 1.27)) (justify left))
+    )
+    (property "Footprint" "MountingHole:MountingHole_2.2mm_M2" (id 2) (at 257.81 234.95 0)
+      (effects (font (size 1.27 1.27)) hide)
+    )
+    (property "Datasheet" "~" (id 3) (at 257.81 234.95 0)
+      (effects (font (size 1.27 1.27)) hide)
+    )
   )
   (symbol (lib_id "power:GND") (at 109.22 175.26 0) (unit 1)
@@
     (pin "9")
   )
+  (symbol (lib_id "Mechanical:MountingHole") (at 257.81 229.87 0) (unit 1)
+    (in_bom yes) (on_board yes)
+    (property "Reference" "H1" (id 0) (at 252.73 229.87 0)
+      (effects (font (size 1.27 1.27)) (justify left))
+    )
+    (property "Value" "MountingHole" (id 1) (at 260.35 229.87 0)
+      (effects (font (size 1.27 1.27)) (justify left))
+    )
+    (property "Footprint" "MountingHole:MountingHole_2.2mm_M2" (id 2) (at 257.81 229.87 0)
+      (effects (font (size 1.27 1.27)) hide)
+    )
+    (property "Datasheet" "~" (id 3) (at 257.81 229.87 0)
+      (effects (font (size 1.27 1.27)) hide)
+    )
+  )
   (symbol (lib_id "power:GND") (at 184.15 153.67 0) (unit 1)
     (in_bom yes) (on_board yes) (fields_autoplaced)
@@
     )
     (pin "1")
+  )
+  (symbol (lib_id "Mechanical:MountingHole") (at 257.81 245.11 0) (unit 1)
+    (in_bom yes) (on_board yes)
+    (property "Reference" "H4" (id 0) (at 252.73 245.11 0)
+      (effects (font (size 1.27 1.27)) (justify left))
+    )
+    (property "Value" "MountingHole" (id 1) (at 260.35 245.11 0)
+      (effects (font (size 1.27 1.27)) (justify left))
+    )
+    (property "Footprint" "MountingHole:MountingHole_2.2mm_M2" (id 2) (at 257.81 245.11 0)
+      (effects (font (size 1.27 1.27)) hide)
+    )
+    (property "Datasheet" "~" (id 3) (at 257.81 245.11 0)
+      (effects (font (size 1.27 1.27)) hide)
+    )
   )
   (symbol (lib_id "power:+3.3V") (at 306.07 74.93 270) (unit 1)
@@
       (reference "FB1") (unit 1) (value "120R") (footprint "Inductor_SMD:L_0603_1608Metric")
     )
+    (path "/7af148fc-3a03-4951-af30-8468348243a1"
+      (reference "H1") (unit 1) (value "MountingHole") (footprint "MountingHole:MountingHole_2.2mm_M2")
+    )
+    (path "/56e1cf0e-d61b-4dfe-8d76-cf4629de505d"
+      (reference "H2") (unit 1) (value "MountingHole") (footprint "MountingHole:MountingHole_2.2mm_M2")
+    )
+    (path "/068537eb-19b5-43c2-a1fa-b0fc53cc0414"
+      (reference "H3") (unit 1) (value "MountingHole") (footprint "MountingHole:MountingHole_2.2mm_M2")
+    )
+    (path "/82dedc1f-8f46-4680-98a3-56f743ddceb7"
+      (reference "H4") (unit 1) (value "MountingHole") (footprint "MountingHole:MountingHole_2.2mm_M2")
+    )
     (path "/14507397-e49c-4710-acf9-dbb3fde324ae"

Commit message: signal routing
Connections:
- net PA15: now also J2.6 (Pin_6)
- net PB3: now also J2.7 (Pin_7); no longer J2.6 (Pin_6)
- net PB4: now also J2.8 (Pin_8); no longer J2.7 (Pin_7)
- net PB5: now also J2.9 (Pin_9); no longer J2.8 (Pin_8)
- net PB6: now also J2.10 (Pin_10); no longer J2.9 (Pin_9)
- net PB7: now also J2.11 (Pin_11); no longer J2.10 (Pin_10)
- net PB8: now also J2.12 (Pin_12); no longer J2.11 (Pin_11)
- net PB9: now also J2.13 (Pin_13); no longer J2.12 (Pin_12)
Changed lines of the file:
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@@
     (effects (font (size 1.27 1.27)) (justify left bottom))
   )
-  (label "PB9" (at 306.07 102.87 180)
+  (label "PB9" (at 306.07 105.41 180)
     (effects (font (size 1.27 1.27)) (justify right bottom))
   )
@@
   )
   (label "PA8" (at 306.07 82.55 180)
+    (effects (font (size 1.27 1.27)) (justify right bottom))
+  )
+  (label "PA15" (at 306.07 87.63 180)
     (effects (font (size 1.27 1.27)) (justify right bottom))
   )
@@
     (effects (font (size 0.5 0.5)) (justify left bottom))
   )
-  (label "PB6" (at 306.07 95.25 180)
+  (label "PB6" (at 306.07 97.79 180)
     (effects (font (size 1.27 1.27)) (justify right bottom))
   )
@@
     (effects (font (size 1.27 1.27)) (justify left bottom))
   )
-  (label "PB4" (at 306.07 90.17 180)
+  (label "PB4" (at 306.07 92.71 180)
     (effects (font (size 1.27 1.27)) (justify right bottom))
   )
@@
     (effects (font (size 1.27 1.27)) (justify right bottom))
   )
-  (label "PB5" (at 306.07 92.71 180)
+  (label "PB5" (at 306.07 95.25 180)
     (effects (font (size 1.27 1.27)) (justify right bottom))
   )
@@
     (effects (font (size 1.27 1.27)) (justify right bottom))
   )
-  (label "PB3" (at 306.07 87.63 180)
+  (label "PB3" (at 306.07 90.17 180)
     (effects (font (size 1.27 1.27)) (justify right bottom))
   )
-  (label "PB7" (at 306.07 97.79 180)
+  (label "PB7" (at 306.07 100.33 180)
     (effects (font (size 1.27 1.27)) (justify right bottom))
   )
@@
     (effects (font (size 1.27 1.27)) (justify right bottom))
   )
-  (label "PB8" (at 306.07 100.33 180)
+  (label "PB8" (at 306.07 102.87 180)
     (effects (font (size 1.27 1.27)) (justify right bottom))
   )
