File: pcb/stm32_uc.kicad_pcb (KiCad board)
At the start: 2 copper layers, 59 x 31 mm, 32 parts, among them J1 Conn_01x18_Male, J2 Conn_01x18_Male, J3 USB_C_Receptacle_USB2.0, J4 Conn_01x04_Male, SW1 SW_SPDT, U1 AMS1117-3.3, U2 STM32F103C8T6, Y1 16Mhz

Commit message: more signal routing, started power routing
Parts:
- moved C1 0.27 mm to (182.1, 108.0)
Routing:
- net /PB14: track 0.00 -> 18.8 mm, vias 0 -> 2
- net /PB13: track 0.00 -> 16.0 mm
- net /PB12: track 0.00 -> 13.4 mm
- net GND: track 31.0 -> 32.2 mm, vias 6 -> 13
- added copper zone on F.Cu, net +3V3
- added copper zone on F.Cu, net GND
- added copper zone on F.Cu, net VBUS
Changed lines of the file:
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@@
     (property "Sheetname" "")
     (attr smd)
-    (fp_text reference "C2" (at 3 0) (layer "F.SilkS")
+    (fp_text reference "C2" (at -2.7 0.05) (layer "F.SilkS")
       (effects (font (size 1 1) (thickness 0.15)))
     )
@@
   )
   (footprint "Capacitor_SMD:C_0805_2012Metric" (layer "F.Cu")
-    (at 182 107.75 -90)
+    (at 182.1 108 -90)
     (descr "Capacitor SMD 0805 (2012 Metric), square (rectangular) end terminal, IPC_7351 nominal, (Body size source: IPC-SM-782 page 76, https://www.pcb-3d.com/wordpress/wp-content/uploads/ipc-sm-782a_amendment_1_and_2.pdf, https://docs.google.com/spreadsheets/d/1BsfQQcO9C6DZCsRaXUlFlo91Tg2WpOkGARC1WS5S8t0/edit?usp=sharing), generated with kicad-footprint-generator")
     (tags "capacitor")
@@
     (property "Sheetname" "")
     (attr smd)
-    (fp_text reference "C1" (at 2.5 0 180) (layer "F.SilkS")
+    (fp_text reference "C1" (at -2.35 0 180) (layer "F.SilkS")
       (effects (font (size 1 1) (thickness 0.15)))
     )
@@
   (segment (start 139.82 114.72) (end 139.8 114.7) (width 0.5) (layer "F.Cu") (net 2))
   (segment (start 155.096 104.937) (end 154.554489 105.478511) (width 0.3) (layer "F.Cu") (net 2))
+  (segment (start 162.55 97.85) (end 162.55 99.6625) (width 0.3) (layer "F.Cu") (net 2))
   (segment (start 179.24 104.25) (end 178.15 104.25) (width 0.5) (layer "F.Cu") (net 2))
   (segment (start 158.704 100.249) (end 158.2075 100.249) (width 0.5) (layer "F.Cu") (net 2))
   (segment (start 160.6375 104.575) (end 158.49 104.575) (width 0.3) (layer "F.Cu") (net 2))
+  (segment (start 162.5 97.8) (end 162.55 97.85) (width 0.3) (layer "F.Cu") (net 2))
   (segment (start 153.406 108.933) (end 153.434 108.905) (width 0.3) (layer "F.Cu") (net 2))
   (segment (start 158.49 104.575) (end 158.45 104.615) (width 0.3) (layer "F.Cu") (net 2))
   (segment (start 178.15 104.25) (end 178.1 104.2) (width 0.5) (layer "F.Cu") (net 2))
-  (segment (start 162.55 99.6625) (end 162.55 97.85) (width 0.3) (layer "F.Cu") (net 2))
-  (segment (start 162.55 100.75) (end 163 101.2) (width 0.3) (layer "F.Cu") (net 2))
+  (segment (start 171.783 101.483) (end 171.8 101.5) (width 0.3) (layer "F.Cu") (net 2))
   (segment (start 142.334997 93.765003) (end 142.3 93.8) (width 0.5) (layer "F.Cu") (net 2))
   (segment (start 142.334997 91.499995) (end 142.334997 93.765003) (width 0.5) (layer "F.Cu") (net 2))
@@
   (segment (start 167.05 107.9875) (end 167.05 109.411) (width 0.3) (layer "F.Cu") (net 2))
   (segment (start 151.706 104.529) (end 151.706 104.429) (width 0.3) (layer "F.Cu") (net 2))
-  (segment (start 162.55 99.6625) (end 162.55 100.75) (width 0.3) (layer "F.Cu") (net 2))
   (segment (start 139.794997 91.499995) (end 142.334997 91.499995) (width 0.5) (layer "F.Cu") (net 2))
   (segment (start 170.55 101.575) (end 168.9625 101.575) (width 0.3) (layer "F.Cu") (net 2))
   (segment (start 167.05 106.45) (end 167 106.4) (width 0.3) (layer "F.Cu") (net 2))
   (segment (start 185.99 98.5) (end 185.99 97.41) (width 0.5) (layer "F.Cu") (net 2))
-  (segment (start 162.55 99.6625) (end 162.54952 99.66202) (width 0.3) (layer "F.Cu") (net 2))
+  (segment (start 162.55 99.6625) (end 162.55 100.75) (width 0.3) (layer "F.Cu") (net 2))
+  (segment (start 170.642 101.483) (end 171.783 101.483) (width 0.3) (layer "F.Cu") (net 2))
   (segment (start 139.82 117) (end 139.82 114.72) (width 0.5) (layer "F.Cu") (net 2))
   (segment (start 158.2075 100.249) (end 156.3875 98.429) (width 0.5) (layer "F.Cu") (net 2))
@@
   (segment (start 170.642 101.483) (end 170.55 101.575) (width 0.3) (layer "F.Cu") (net 2))
   (segment (start 153.406 110.429) (end 153.406 108.933) (width 0.3) (layer "F.Cu") (net 2))
+  (segment (start 162.55 100.75) (end 163 101.2) (width 0.3) (layer "F.Cu") (net 2))
   (segment (start 154.554489 105.478511) (end 152.655511 105.478511) (width 0.3) (layer "F.Cu") (net 2))
   (segment (start 155.096 101.579) (end 154.056 101.579) (width 0.3) (layer "F.Cu") (net 2))
-  (segment (start 162.55 97.85) (end 162.5 97.8) (width 0.3) (layer "F.Cu") (net 2))
   (segment (start 185.99 97.41) (end 186 97.4) (width 0.5) (layer "F.Cu") (net 2))
+  (via (at 181.6 110.2) (size 0.8) (drill 0.4) (layers "F.Cu" "B.Cu") (free) (net 2))
   (via (at 167 106.4) (size 0.8) (drill 0.4) (layers "F.Cu" "B.Cu") (net 2))
   (via (at 163 101.2) (size 0.8) (drill 0.4) (layers "F.Cu" "B.Cu") (net 2))
+  (via (at 178.8 113.3) (size 0.8) (drill 0.4) (layers "F.Cu" "B.Cu") (free) (net 2))
   (via (at 139.8 114.7) (size 0.8) (drill 0.4) (layers "F.Cu" "B.Cu") (net 2))
+  (via (at 178.8 114.3) (size 0.8) (drill 0.4) (layers "F.Cu" "B.Cu") (free) (net 2))
+  (via (at 182.7 110.2) (size 0.8) (drill 0.4) (layers "F.Cu" "B.Cu") (free) (net 2))
   (via (at 142.3 93.8) (size 0.8) (drill 0.4) (layers "F.Cu" "B.Cu") (net 2))
+  (via (at 171.8 101.5) (size 0.8) (drill 0.4) (layers "F.Cu" "B.Cu") (net 2))
+  (via (at 177.7 111.8) (size 0.8) (drill 0.4) (layers "F.Cu" "B.Cu") (free) (net 2))
   (via (at 178.1 104.2) (size 0.8) (drill 0.4) (layers "F.Cu" "B.Cu") (net 2))
+  (via (at 177.7 110.9) (size 0.8) (drill 0.4) (layers "F.Cu" "B.Cu") (free) (net 2))
   (via (at 186 97.4) (size 0.8) (drill 0.4) (layers "F.Cu" "B.Cu") (net 2))
   (segment (start 158.838 101.075) (end 160.6375 101.075) (width 0.3) (layer "F.Cu") (net 3))
@@
   (segment (start 166.55 107.9875) (end 166.55 110.71) (width 0.3) (layer "F.Cu") (net 9))
   (segment (start 166.55 110.71) (end 172.84 117) (width 0.3) (layer "F.Cu") (net 9))
+  (segment (start 175.38 117) (end 170.6 112.22) (width 0.3) (layer "F.Cu") (net 10))
+  (segment (start 169.475 106.575) (end 168.9625 106.575) (width 0.3) (layer "F.Cu") (net 10))
+  (segment (start 170.6 112.22) (end 170.6 107.7) (width 0.3) (layer "F.Cu") (net 10))
+  (segment (start 170.6 107.7) (end 169.475 106.575) (width 0.3) (layer "F.Cu") (net 10))
+  (segment (start 169.800361 106.075) (end 168.9625 106.075) (width 0.3) (layer "F.Cu") (net 11))
+  (segment (start 177.92 117) (end 176.720489 115.800489) (width 0.3) (layer "F.Cu") (net 11))
+  (segment (start 171.09952 111.59952) (end 171.09952 107.374159) (width 0.3) (layer "F.Cu") (net 11))
+  (segment (start 175.300489 115.800489) (end 171.09952 111.59952) (width 0.3) (layer "F.Cu") (net 11))
+  (segment (start 171.09952 107.374159) (end 169.800361 106.075) (width 0.3) (layer "F.Cu") (net 11))
+  (segment (start 176.720489 115.800489) (end 175.300489 115.800489) (width 0.3) (layer "F.Cu") (net 11))
+  (segment (start 171.275 105.575) (end 168.9625 105.575) (width 0.3) (layer "F.Cu") (net 12))
+  (segment (start 180.46 117) (end 180.46 114.64) (width 0.3) (layer "F.Cu") (net 12))
+  (segment (start 180.46 114.64) (end 180.5 114.6) (width 0.3) (layer "F.Cu") (net 12))
+  (segment (start 171.7 106) (end 171.275 105.575) (width 0.3) (layer "F.Cu") (net 12))
+  (via (at 180.5 114.6) (size 0.8) (drill 0.4) (layers "F.Cu" "B.Cu") (net 12))
+  (via (at 171.7 106) (size 0.8) (drill 0.4) (layers "F.Cu" "B.Cu") (net 12))
+  (segment (start 180.5 112.64003) (end 173.85997 106) (width 0.3) (layer "B.Cu") (net 12))
+  (segment (start 173.85997 106) (end 171.7 106) (width 0.3) (layer "B.Cu") (net 12))
+  (segment (start 180.5 114.6) (end 180.5 112.64003) (width 0.3) (layer "B.Cu") (net 12))
   (segment (start 168.9625 105.075) (end 173.825 105.075) (width 0.3) (layer "F.Cu") (net 13))
   (segment (start 173.825 105.075) (end 175.1 103.8) (width 0.3) (layer "F.Cu") (net 13))
@@
   (segment (start 185.064259 105) (end 184.925 105) (width 0.3) (layer "F.Cu") (net 50))
   (segment (start 186.275 104.15) (end 185.914259 104.15) (width 0.3) (layer "F.Cu") (net 50))
+  (zone (net 3) (net_name "+3V3") (layer "F.Cu") (hatch edge 0.508)
+    (connect_pads yes (clearance 0.3))
+    (min_thickness 0.25) (filled_areas_thickness no)
+    (fill yes (thermal_gap 0.508) (thermal_bridge_width 0.508))
+    (polygon
+      (pts
+        (xy 178.2 108.1)
+        (xy 180.4 108.1)
+        (xy 180.6 108.3)
+        (xy 180.6 109.8)
+        (xy 180.4 110)
+        (xy 178.1 110)
+        (xy 177.2 110)
+        (xy 176.2 111)
+        (xy 176.2 114.4)
+        (xy 175.9 114.7)
+        (xy 175.2 114.7)
+        (xy 174.8 114.3)
+        (xy 174.8 111.6)
+        (xy 174.4 111.2)
+        (xy 172.1 111.2)
+        (xy 171.7 110.8)
+        (xy 171.7 107.3)
+        (xy 172.2 106.8)
+        (xy 176.9 106.8)
+      )
+    )
+  )
+  (zone (net 1) (net_name "VBUS") (layer "F.Cu") (hatch edge 0.508)
+    (connect_pads yes (clearance 0.3))
+    (min_thickness 0.25) (filled_areas_thickness no)
+    (fill yes (thermal_gap 0.508) (thermal_bridge_width 0.508))
+    (polygon
+      (pts
+        (xy 183.2 106.3)
+        (xy 186.7 106.3)
+        (xy 186.9 106.5)
+        (xy 186.9 106.9)
+        (xy 186.7 107.1)
+        (xy 184.2 107.1)
+        (xy 183.5 107.8)
+        (xy 178.5 107.8)
+        (xy 178 107.3)
+        (xy 178 105.8)
+        (xy 178.4 105.5)
+        (xy 182.4 105.5)
+      )
+    )
+  )
+  (zone (net 2) (net_name "GND") (layer "F.Cu") (hatch edge 0.508)
+    (connect_pads yes (clearance 0.3))
+    (min_thickness 0.25) (filled_areas_thickness no)
+    (fill yes (thermal_gap 0.508) (thermal_bridge_width 0.508))
+    (polygon
+      (pts
+        (xy 183.3 108.4)
+        (xy 183.3 110.7)
+        (xy 183 111)
+        (xy 181.3 111)
+        (xy 181 111.3)
+        (xy 181 112.6)
+        (xy 180.6 113)
+        (xy 179.8 113)
+        (xy 179.5 113.3)
+        (xy 179.5 114.5)
+        (xy 179.1 114.9)
+        (xy 176.9 114.9)
+        (xy 176.6 114.6)
+        (xy 176.6 112.3)
+        (xy 177 111.9)
+        (xy 177 110.8)
+        (xy 177.5 110.3)
+        (xy 180.6 110.3)
+        (xy 180.9 110)
+        (xy 180.9 108.5)
+        (xy 181.3 108.1)
+        (xy 183 108.1)
+      )
+    )
+  )
   (zone (net 2) (net_name "GND") (layer "B.Cu") (name "gndplane") (hatch edge 0.508)
     (connect_pads (clearance 0.3))

Commit message: finished routing
Parts:
- moved C11 17.3 mm to (168.5, 96.3), turned to 90 degrees
- moved R1 0.62 mm to (143.6, 106.6)
- moved D1 0.61 mm to (144.4, 104.6), turned to 0 degrees
Routing:
- net +3V3: track 14.5 -> 159.0 mm, vias 0 -> 10
- net /BOOT0: track 0.00 -> 28.9 mm, vias 0 -> 2
- net /PA1: track 0.00 -> 28.6 mm, vias 0 -> 1
- net /PA0: track 0.00 -> 28.2 mm, vias 0 -> 1
- net /PC15: track 0.00 -> 23.1 mm, vias 0 -> 1
- net /PC14: track 0.00 -> 18.3 mm
- net /PA2: track 0.00 -> 17.7 mm
- net /PC13: track 0.00 -> 17.6 mm, vias 0 -> 1
- net unconnected-(J3-PadS1): track 0.00 -> 15.4 mm
- net /NRST: track 0.00 -> 12.8 mm, vias 0 -> 2
- net VBUS: track 1.35 -> 9.15 mm, vias 0 -> 1
- net GND: track 32.2 -> 39.8 mm, vias 13 -> 19
- net +3.3VA: track 3.90 -> 8.26 mm
- net /SW_BOOT0: track 0.00 -> 3.10 mm
- net /PB15: track 20.1 -> 21.7 mm
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